Commit message: added the gripper
added the visuals, no physics

File: Kinova-DT-Project/Assets/Kinova URDF/gen3_robotiq_2f_85.urdf (robot description, URDF)
Before this commit: robot gen3_robotiq_2f_85, 23 links, 22 joints
Links:
- removed link left_inner_finger_pad
- removed link right_inner_finger_pad
- removed link robotiq_arg2f_base_link
- added link robotiq_85_base_link, mass 0.30915; collision mesh filename=package://kortex_description/gripper_test/meshes/robotiq_85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; visual mesh filename=package://kortex_description/gripper_test/meshes/robotiq_85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
- link left_inner_finger: mass 0.0104003125914103 -> 0.00724255346165745; geometry collision mesh filename=package://kortex_description/gripper_test/meshes/inner_fing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; visual mesh filename=package://kortex_description/gripper_test/meshes/inner_fing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
- link left_inner_knuckle: mass 0.0271177346495152 -> 0.0110930853895903; geometry collision mesh filename=package://kortex_description/gripper_test/meshes/inner_knuc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; visual mesh filename=package://kortex_description/gripper_test/meshes/inner_knuc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
- link left_outer_finger: mass 0.022614240507152 -> 0.0273093985570947; geometry collision mesh filename=package://kortex_description/gripper_test/meshes/outer_fing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; visual mesh filename=package://kortex_description/gripper_test/meshes/outer_fing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
- link left_outer_knuckle: mass 0.00853198276973456 -> 0.00684838849434396; geometry collision mesh filename=package://kortex_description/gripper_test/meshes/outer_knuc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; visual mesh filename=package://kortex_description/gripper_test/meshes/outer_knuc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
- link right_inner_finger: mass 0.0104003125914103 -> 0.00724255346165744; geometry collision mesh filename=package://kortex_description/gripper_test/meshes/inner_fing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; visual mesh filename=package://kortex_description/gripper_test/meshes/inner_fing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
- link right_inner_knuckle: mass 0.0271177346495152 -> 0.0110930853895903; geometry collision mesh filename=package://kortex_description/gripper_test/meshes/inner_knuc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; visual mesh filename=package://kortex_description/gripper_test/meshes/inner_knuc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
- link right_outer_finger: mass 0.022614240507152 -> 0.0273093985570947; geometry collision mesh filename=package://kortex_description/gripper_test/meshes/outer_fing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; visual mesh filename=package://kortex_description/gripper_test/meshes/outer_fing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
- link right_outer_knuckle: mass 0.00853198276973456 -> 0.00684838849401352; geometry collision mesh filename=package://kortex_description/gripper_test/meshes/outer_knuc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; visual mesh filename=package://kortex_description/gripper_test/meshes/outer_knuc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
Joints:
- removed joint finger_joint
- removed joint gripper_base_joint
- removed joint left_inner_finger_pad_joint
- removed joint right_inner_finger_pad_joint
- added joint left_outer_knuckle_joint: type revolute, parent robotiq_85_base_link, child left_outer_knuckle, origin xyz=0.0306011444260539 0 0.0627920162695395 rpy=0 0 0, axis 0 -1 0, limit lower=-0.8757 upper=0.8757 effort=1000 velocity=2.0
- added joint robotiq_85_base_joint: type fixed, parent EndEffector_Link, child robotiq_85_base_link, origin xyz=0 0 0 rpy=0 0 0
- joint left_inner_finger_joint: axis 1 0 0 -> 0 -1 0; mimic joint=finger_joint multiplier=-1 offset=0 -> (none); origin xyz=0 0.0061 0.0471 rpy=0 0 0 -> xyz=0.034585310861294 0 0.0454970193817975 rpy=0 0 0; parent left_outer_finger -> left_inner_knuckle
- joint left_inner_knuckle_joint: axis 1 0 0 -> 0 -1 0; limit lower=0 upper=0.8757 effort=1000 velocity=2.0 -> lower=-0.8757 upper=0.8757 effort=1000 velocity=2.0; mimic joint=finger_joint multiplier=1 offset=0 -> (none); origin xyz=0 -0.0127 0.06142 rpy=0 0 3.141592653589793 -> xyz=0.0127000000001501 0 0.0693074999999639 rpy=0 0 0; parent robotiq_arg2f_base_link -> robotiq_85_base_link
- joint left_outer_finger_joint: axis 1 0 0 -> 0 -1 0; origin xyz=0 0.0315 -0.0041 rpy=0 0 0 -> xyz=0.0316910442266543 0 -0.00193396375724605 rpy=0 0 0
- joint right_inner_finger_joint: axis 1 0 0 -> 0 1 0; mimic joint=finger_joint multiplier=-1 offset=0 -> (none); origin xyz=0 0.0061 0.0471 rpy=0 0 0 -> xyz=0.0341060475457406 0 0.0458573878541688 rpy=0 0 0; parent right_outer_finger -> right_inner_knuckle
- joint right_inner_knuckle_joint: axis 1 0 0 -> 0 1 0; limit lower=0 upper=0.8757 effort=1000 velocity=2.0 -> lower=-0.8757 upper=0.8757 effort=1000 velocity=2.0; mimic joint=finger_joint multiplier=1 offset=0 -> (none); origin xyz=0 0.0127 0.06142 rpy=0 0 0.0 -> xyz=-0.0126999999998499 0 0.0693075000000361 rpy=0 0 3.14159265358979; parent robotiq_arg2f_base_link -> robotiq_85_base_link
- joint right_outer_finger_joint: axis 1 0 0 -> 0 1 0; origin xyz=0 0.0315 -0.0041 rpy=0 0 0 -> xyz=0.0317095909367246 0 -0.0016013564954687 rpy=0 0 0
- joint right_outer_knuckle_joint: axis 1 0 0 -> 0 1 0; limit lower=0 upper=0.81 effort=1000 velocity=2.0 -> lower=-0.8757 upper=0.8757 effort=1000 velocity=2.0; mimic joint=finger_joint multiplier=1 offset=0 -> (none); origin xyz=0 0.0306011 0.054904 rpy=0 0 0 -> xyz=-0.0306011444258893 0 0.0627920162695395 rpy=0 0 3.14159265358979; parent robotiq_arg2f_base_link -> robotiq_85_base_link
