Commit message: files sorting

File: Kinova-DT-Project/Assets/Kinova URDF/robotiq_arg85_description.URDF (robot description, URDF)
Before this commit: robot robotiq_arg2f_85_model, 9 links, 9 joints
Joints:
- removed joint left_outer_knuckle_joint
- removed joint robotiq_85_base_joint
- added joint finger_joint: type revolute, parent robotiq_85_base_link, child left_outer_knuckle, origin xyz=0.0306011444260539 0 0.0627920162695395 rpy=0 0 0, axis 0 -1 0, limit lower=0 upper=0.725 effort=1000 velocity=2.0
- joint left_inner_finger_joint: limit lower=-0.8757 upper=0.8757 effort=1000 velocity=2.0 -> lower=0 upper=0.8757 effort=1000 velocity=2.0; mimic (none) -> joint=finger_joint multiplier=-1 offset=0
- joint left_inner_knuckle_joint: limit lower=-0.8757 upper=0.8757 effort=1000 velocity=2.0 -> lower=0 upper=0.8757 effort=1000 velocity=2.0; mimic (none) -> joint=finger_joint multiplier=1 offset=0
- joint right_inner_finger_joint: limit lower=-0.8757 upper=0.8757 effort=1000 velocity=2.0 -> lower=0 upper=0.8757 effort=1000 velocity=2.0; mimic (none) -> joint=finger_joint multiplier=1 offset=0
- joint right_inner_knuckle_joint: limit lower=-0.8757 upper=0.8757 effort=1000 velocity=2.0 -> lower=0 upper=0.8757 effort=1000 velocity=2.0; mimic (none) -> joint=finger_joint multiplier=-1 offset=0
- joint right_outer_knuckle_joint: limit lower=-0.8757 upper=0.8757 effort=1000 velocity=2.0 -> lower=0 upper=0.8757 effort=1000 velocity=2.0; mimic (none) -> joint=finger_joint multiplier=-1 offset=0
